Commit message: Modified controller to publish propirtional, integral and derivative errors. Added plots from step response tests in the Images folder.

File: CPR_project/my_1dof_robot/urdf/my_1dof_robot.urdf (robot description, URDF)
Before this commit: robot my_1dof_robot, 3 links, 2 joints
Joints:
- joint joint_1: limit lower=-3.14 upper=3.14 effort=100 velocity=3.14 -> lower=-3.14 upper=3.14 effort=1000 velocity=3.14

Commit message: Modified 1dof controller gains. Modified pendulum actuators saturation limits.

File: CPR_project/my_1dof_robot/urdf/my_1dof_robot.urdf (robot description, URDF)
Before this commit: robot my_1dof_robot, 3 links, 2 joints
Joints:
- joint joint_1: limit lower=-3.14 upper=3.14 effort=1000 velocity=3.14 -> lower=-3.14 upper=3.14 effort=100 velocity=100
