Commit message: Created simple pendulum robot my_1dof_robot. Added par_computado_1dof controller (for now it is a PID, to be modified to become par computado on 1 joint). Moved .stl meshes inside irb120 eliminating dependency on external packages. Unified .launch file into my_moveit_gazebo.launch.

File: CPR_project/irb120/urdf/irb120.urdf (robot description, URDF)
Before this commit: robot abb_irb120_model, 10 links, 9 joints
Links:
- link base_link: geometry collision mesh filename=package://irb120/meshes/visual/base_link.stl; visual mesh filename=package://irb120/meshes/visual/base_link.stl
- link link_1: geometry collision mesh filename=package://irb120/meshes/visual/link_1.stl; visual mesh filename=package://irb120/meshes/visual/link_1.stl
- link link_2: geometry collision mesh filename=package://irb120/meshes/visual/link_2.stl; visual mesh filename=package://irb120/meshes/visual/link_2.stl
- link link_3: geometry collision mesh filename=package://irb120/meshes/visual/link_3.stl; visual mesh filename=package://irb120/meshes/visual/link_3.stl
- link link_4: geometry collision mesh filename=package://irb120/meshes/visual/link_4.stl; visual mesh filename=package://irb120/meshes/visual/link_4.stl
- link link_5: geometry collision mesh filename=package://irb120/meshes/visual/link_5.stl; visual mesh filename=package://irb120/meshes/visual/link_5.stl
- link link_6: geometry collision mesh filename=package://irb120/meshes/visual/link_6.stl; visual mesh filename=package://irb120/meshes/visual/link_6.stl

Commit message: Implemented the calculation of dynamics matrices in par_computado_6dof using KDL library. Added publishers for datalogging to par_computado_6dof.

File: CPR_project/irb120/urdf/irb120.urdf (robot description, URDF)
Before this commit: robot abb_irb120_model, 10 links, 9 joints
Joints:
- joint joint_1: limit lower=-2.87979 upper=2.87979 effort=30 velocity=4.36332 -> lower=-2.87979 upper=2.87979 effort=100 velocity=4.36332
- joint joint_2: limit lower=-1.91986 upper=1.91986 effort=30 velocity=4.36332 -> lower=-1.91986 upper=1.91986 effort=100 velocity=4.36332
- joint joint_3: limit lower=-1.91986 upper=1.22173 effort=30 velocity=4.36332 -> lower=-1.91986 upper=1.22173 effort=100 velocity=4.36332
- joint joint_4: limit lower=-2.79253 upper=2.79253 effort=30 velocity=5.58505 -> lower=-2.79253 upper=2.79253 effort=100 velocity=5.58505
- joint joint_5: limit lower=-2.094395 upper=2.094395 effort=30 velocity=5.58505 -> lower=-2.094395 upper=2.094395 effort=100 velocity=5.58505
- joint joint_6: limit lower=-6.98132 upper=6.98132 effort=30 velocity=7.33038 -> lower=-6.98132 upper=6.98132 effort=100 velocity=7.33038

Commit message: Modified comments

File: CPR_project/irb120/urdf/irb120.urdf (robot description, URDF)
Before this commit: robot abb_irb120_model, 10 links, 9 joints
Joints:
- joint joint_1: limit lower=-2.87979 upper=2.87979 effort=100 velocity=4.36332 -> lower=-2.87979 upper=2.87979 effort=200 velocity=4.36332
- joint joint_2: limit lower=-1.91986 upper=1.91986 effort=100 velocity=4.36332 -> lower=-1.91986 upper=1.91986 effort=200 velocity=4.36332
- joint joint_3: limit lower=-1.91986 upper=1.22173 effort=100 velocity=4.36332 -> lower=-1.91986 upper=1.22173 effort=200 velocity=4.36332
- joint joint_4: limit lower=-2.79253 upper=2.79253 effort=100 velocity=5.58505 -> lower=-2.79253 upper=2.79253 effort=200 velocity=5.58505
- joint joint_5: limit lower=-2.094395 upper=2.094395 effort=100 velocity=5.58505 -> lower=-2.094395 upper=2.094395 effort=200 velocity=5.58505
- joint joint_6: limit lower=-6.98132 upper=6.98132 effort=100 velocity=7.33038 -> lower=-6.98132 upper=6.98132 effort=200 velocity=7.33038
